Commit message: Removed the laser scanner to ease the computational load for my MC trials.

File: p3dx_description/urdf/pioneer3dx.xacro (robot description, xacro)
@@ -169,5 +169,5 @@
 	<xacro:p3dx_wheel suffix="left" parent="base_link" reflect="1"/>
 	<xacro:p3dx_wheel suffix="right" parent="base_link" reflect="-1"/>
-  <!-- front_sonar -->
+  <!-- front_sonar >
 	<link name="front_sonar">
 		<inertial>
@@ -196,6 +196,6 @@
 		<parent link="base_link" />
 		<child link="front_sonar" />
-	</joint>
-	<!-- lms100 laser -->
+	</joint-->
+	<!-- lms100 laser >
 	<link name="lms100">
 		<inertial>
@@ -222,4 +222,4 @@
 		<parent link="base_link" />
 		<child link="lms100" />
-	</joint>
+	</joint-->
 </robot>
